Commit message: Change model colors and base size

File: urdf/furuta_pendulum.urdf.xacro (robot description, xacro)
@@ -1,14 +1,8 @@
 <?xml version="1.0"?>
 <robot name="furuta_pendulum" xmlns:xacro="http://www.ros.org/wiki/xacro">
-  <material name="red">
-    <color rgba="1.0 0.0 0.0 1.0" />
+  <material name="grey">
+    <color rgba="0.4 0.4 0.4 1.0" />
   </material>
-  <material name="blue">
-    <color rgba="0.0 0.0 1.0 1.0" />
-  </material>
-  <material name="green">
-    <color rgba="0.0 1.0 0.0 1.0" />
-  </material>
-  <xacro:property name="base_radius" value="0.02" />
+  <xacro:property name="base_radius" value="0.1" />
   <xacro:property name="base_length" value="0.1" />
   <xacro:property name="arm1_radius" value="0.02" />
@@ -22,9 +16,9 @@
         <cylinder radius="${base_radius}" length="${base_length}" />
       </geometry>
-      <material name="red" />
+      <material name="grey" />
     </visual>
   </link>
   <joint name="joint1" type="continuous">
-    <origin xyz="0.0 0.0 ${base_length}" rpy="0.0 0.0 0.0" />
+    <origin xyz="0.0 0.0 ${base_length+arm1_radius}" rpy="0.0 0.0 0.0" />
     <parent link="base_link" />
     <child link="arm1" />
@@ -37,5 +31,5 @@
         <cylinder radius="${arm1_radius}" length="${arm1_length}" />
       </geometry>
-      <material name="blue" />
+      <material name="grey" />
     </visual>
   </link>
@@ -53,5 +47,5 @@
         <cylinder radius="${arm2_radius}" length="${arm2_length}" />
       </geometry>
-      <material name="green" />
+      <material name="grey" />
     </visual>
   </link>

Commit message: Add simulation properties to urdf

File: urdf/furuta_pendulum.urdf.xacro (robot description, xacro)
@@ -1,13 +1,28 @@
 <?xml version="1.0"?>
 <robot name="furuta_pendulum" xmlns:xacro="http://www.ros.org/wiki/xacro">
+  <xacro:arg name="m1" default="0.0" />
+  <xacro:arg name="m2" default="0.0" />
+  <xacro:arg name="l1" default="0.0" />
+  <xacro:arg name="l2" default="0.0" />
+  <xacro:arg name="L1" default="0.0" />
+  <xacro:arg name="L2" default="0.0" />
+  <xacro:arg name="J1" default="0.0" />
+  <xacro:arg name="J2" default="0.0" />
+  <xacro:arg name="b1" default="0.0" />
+  <xacro:arg name="b2" default="0.0" />
   <material name="grey">
-    <color rgba="0.4 0.4 0.4 1.0" />
+    <color rgba="0.8 0.8 0.8 1.0" />
   </material>
   <xacro:property name="base_radius" value="0.1" />
   <xacro:property name="base_length" value="0.1" />
   <xacro:property name="arm1_radius" value="0.02" />
-  <xacro:property name="arm1_length" value="0.278" />
+  <xacro:property name="arm1_length" value="$(arg L1)" />
   <xacro:property name="arm2_radius" value="0.02" />
-  <xacro:property name="arm2_length" value="0.3" />
+  <xacro:property name="arm2_length" value="$(arg L2)" />
+  <!-- https://www.hindawi.com/journals/jcse/2011/528341/ here this inertias
+    are approximated by 0.0, I set them to really low value, to get correct
+    visualtizations in rviz -->
+  <xacro:property name="arm1_inertia_x" value="0.000001" />
+  <xacro:property name="arm2_inertia_z" value="0.000001" />
   <link name="base_link">
     <visual>
@@ -24,4 +39,5 @@
     <child link="arm1" />
     <axis xyz="0 0 1" />
+    <dynamics damping="$(arg b1)" />
   </joint>
   <link name="arm1">
@@ -33,4 +49,17 @@
       <material name="grey" />
     </visual>
+    <collision>
+      <origin xyz="${arm1_length/2.0} 0.0 0.0" rpy="0.0 ${pi/2.0} 0.0" />
+      <geometry>
+        <cylinder radius="${arm1_radius}" length="${arm1_length}" />
+      </geometry>
+    </collision>
+    <inertial>
+      <mass value="$(arg m1)" />
+      <origin xyz="$(arg l1) 0.0 0.0" rpy="0.0 0.0 0.0" />
+      <inertia ixx="${arm1_inertia_x}" ixy="0.0"       ixz="0.0"
+                                       iyy="$(arg J1)" iyz="0.0"
+                                                       izz="$(arg J1)" />
+    </inertial>
   </link>
   <joint name="joint2" type="continuous">
@@ -40,4 +69,5 @@
     <child link="arm2" />
     <axis xyz="1 0 0" />
+    <dynamics damping="$(arg b2)" />
   </joint>
   <link name="arm2">
@@ -49,4 +79,17 @@
       <material name="grey" />
     </visual>
+    <collision>
+      <origin xyz="0.0 0.0 ${arm2_length/2.0}" rpy="0.0 0.0 0.0" />
+      <geometry>
+        <cylinder radius="${arm2_radius}" length="${arm2_length}" />
+      </geometry>
+    </collision>
+    <inertial>
+      <mass value="$(arg m2)" />
+      <origin xyz="0.0 0.0 $(arg l2)" rpy="0.0 0.0 0.0" />
+      <inertia ixx="$(arg J2)" ixy="0.0"       ixz="0.0"
+                               iyy="$(arg J2)" iyz="0.0"
+                                               izz="${arm2_inertia_z}" />
+    </inertial>
   </link>
 </robot>

Commit message: Add ignition simulation

File: urdf/furuta_pendulum.urdf.xacro (robot description, xacro)
@@ -1,4 +1,5 @@
 <?xml version="1.0"?>
 <robot name="furuta_pendulum" xmlns:xacro="http://www.ros.org/wiki/xacro">
+  <xacro:arg name="use_sim" default="true" />
   <xacro:arg name="m1" default="0.0" />
   <xacro:arg name="m2" default="0.0" />
@@ -15,5 +16,6 @@
   </material>
   <xacro:property name="base_radius" value="0.1" />
-  <xacro:property name="base_length" value="0.1" />
+  <xacro:property name="L2" value="$(arg L2)" />
+  <xacro:property name="base_length" value="${L2+0.05}" />
   <xacro:property name="arm1_radius" value="0.02" />
   <xacro:property name="arm1_length" value="$(arg L1)" />
@@ -25,4 +27,12 @@
   <xacro:property name="arm1_inertia_x" value="0.000001" />
   <xacro:property name="arm2_inertia_z" value="0.000001" />
+  <xacro:property name="max_effort" value="4.0" />
+  <xacro:property name="max_velocity" value="15.0" />
+  <link name="world" />
+  <joint name="world_to_base_joint" type="fixed">
+    <origin xyz="0.0 0.0 0.0" rpy="0.0 0.0 0.0" />
+    <parent link="world" />
+    <child link="base_link" />
+  </joint>
   <link name="base_link">
     <visual>
@@ -33,4 +43,17 @@
       <material name="grey" />
     </visual>
+    <collision>
+      <origin xyz="0.0 0.0 ${base_length/2.0}" rpy="0.0 0.0 0.0" />
+      <geometry>
+        <cylinder radius="${base_radius}" length="${base_length}" />
+      </geometry>
+    </collision>
+    <inertial>
+      <mass value="10.0" />
+      <origin xyz="0.0 0.0 0.0" rpy="0.0 0.0 0.0" />
+      <inertia ixx="0.1" ixy="0.0" ixz="0.0"
+        iyy="0.1" iyz="0.0"
+        izz="0.1" />
+    </inertial>
   </link>
   <joint name="joint1" type="continuous">
@@ -40,4 +63,5 @@
     <axis xyz="0 0 1" />
     <dynamics damping="$(arg b1)" />
+    <limit effort="${max_effort}" velocity="${max_velocity}" />
   </joint>
   <link name="arm1">
@@ -58,7 +82,7 @@
       <mass value="$(arg m1)" />
       <origin xyz="$(arg l1) 0.0 0.0" rpy="0.0 0.0 0.0" />
-      <inertia ixx="${arm1_inertia_x}" ixy="0.0"       ixz="0.0"
-                                       iyy="$(arg J1)" iyz="0.0"
-                                                       izz="$(arg J1)" />
+      <inertia ixx="${arm1_inertia_x}" ixy="0.0" ixz="0.0"
+        iyy="$(arg J1)" iyz="0.0"
+        izz="$(arg J1)" />
     </inertial>
   </link>
@@ -70,4 +94,5 @@
     <axis xyz="1 0 0" />
     <dynamics damping="$(arg b2)" />
+    <limit effort="${max_effort}" velocity="${max_velocity}" />
   </joint>
   <link name="arm2">
@@ -88,8 +113,42 @@
       <mass value="$(arg m2)" />
       <origin xyz="0.0 0.0 $(arg l2)" rpy="0.0 0.0 0.0" />
-      <inertia ixx="$(arg J2)" ixy="0.0"       ixz="0.0"
-                               iyy="$(arg J2)" iyz="0.0"
-                                               izz="${arm2_inertia_z}" />
+      <inertia ixx="$(arg J2)" ixy="0.0" ixz="0.0"
+        iyy="$(arg J2)" iyz="0.0"
+        izz="${arm2_inertia_z}" />
     </inertial>
   </link>
+  <ros2_control name="furuta_pendulum" type="system">
+    <hardware>
+      <xacro:if value="$(arg use_sim)">
+        <plugin>ign_ros2_control/IgnitionSystem</plugin>
+      </xacro:if>
+    </hardware>
+    <joint name="joint1">
+      <command_interface name="effort">
+        <param name="min">${-max_effort}</param>
+        <param name="max">${max_effort}</param>
+      </command_interface>
+      <state_interface name="position" />
+      <state_interface name="velocity" />
+    </joint>
+    <joint name="joint2">
+      <command_interface name="effort">
+        <param name="min">${-max_effort}</param>
+        <param name="max">${max_effort}</param>
+      </command_interface>
+      <state_interface name="position" />
+      <state_interface name="velocity" />
+    </joint>
+  </ros2_control>
+  <xacro:if value="$(arg use_sim)">
+    <gazebo>
+      <plugin filename="ign_ros2_control-system"
+        name="ign_ros2_control::IgnitionROS2ControlPlugin">
+        <parameters>$(find furuta_pendulum)/config/furuta_pendulum_ros2_control.yaml</parameters>
+        <ros>
+          <remapping>/forward_effort_controller/commands:=/effort_control</remapping>
+        </ros>
+      </plugin>
+    </gazebo>
+  </xacro:if>
 </robot>
