Commit message: Working lqr with furuta using drake

File: furuta_pendulum_drake/urdf/furuta_pendulum.urdf (robot description, URDF)
Before this commit: robot furuta_pendulum, 4 links, 3 joints
Links:
- link arm1: geometry visual cylinder length=0.278 radius=0.02
- link arm2: geometry visual cylinder length=0.3 radius=0.02
- link base_link: geometry visual cylinder length=0.35 radius=0.1

Commit message: Update drake urdf

File: furuta_pendulum_drake/urdf/furuta_pendulum.urdf (robot description, URDF)
Before this commit: robot furuta_pendulum, 4 links, 3 joints
Links:
- link arm1: mass 0.3 -> 0.040466; geometry visual cylinder length=0.093525 radius=0.005
- link arm2: mass 0.075 -> 0.009801; geometry visual cylinder length=0.129 radius=0.005
- link base_link: geometry visual cylinder length=0.179 radius=0.025
Joints:
- joint joint1: origin xyz=0.0 0.0 0.37 rpy=0.0 0.0 0.0 -> xyz=0.0 0.0 0.184 rpy=0.0 0.0 0.0
- joint joint2: origin xyz=0.278 0.0 0.0 rpy=-3.141592653589793 0.0 0.0 -> xyz=0.093525 0.0 0.0 rpy=-3.141592653589793 0.0 0.0
