Commit message: Change joint names to be consistent with hardware

File: furuta_pendulum_control_toolbox/model/furuta_pendulum.urdf (robot description, URDF)
Before this commit: robot furuta_pendulum, 3 links, 2 joints
Joints:
- removed joint joint2
- added joint joint0: type continuous, parent base_link, child arm1, origin xyz=0.0 0.0 0.184 rpy=0.0 0.0 0.0, axis 0 0 1, limit effort=4.0 velocity=15.0
- joint joint1: axis 0 0 1 -> 1 0 0; child arm1 -> arm2; origin xyz=0.0 0.0 0.184 rpy=0.0 0.0 0.0 -> xyz=0.093525 0.0 0.0 rpy=-3.141592653589793 0.0 0.0; parent base_link -> arm1

File: furuta_pendulum_description/urdf/furuta_pendulum.urdf.xacro (robot description, xacro)
@@ -28,5 +28,6 @@
   <xacro:property name="arm2_inertia_z" value="0.000001" />
   <xacro:property name="max_effort" value="4.0" />
-  <xacro:property name="max_velocity" value="15.0" />
+  <xacro:property name="max_velocity_joint0" value="18.0" />
+  <xacro:property name="max_velocity_joint1" value="100.0" />
   <link name="world" />
   <joint name="world_to_base_joint" type="fixed">
@@ -57,5 +58,5 @@
     </inertial>
   </link>
-  <joint name="joint1" type="continuous">
+  <joint name="joint0" type="continuous">
     <origin xyz="0.0 0.0 ${base_length+arm1_radius}" rpy="0.0 0.0 0.0" />
     <parent link="base_link" />
@@ -63,5 +64,5 @@
     <axis xyz="0 0 1" />
     <dynamics damping="$(arg b1)" />
-    <limit effort="${max_effort}" velocity="${max_velocity}" />
+    <limit effort="${max_effort}" velocity="${max_velocity_joint0}" />
   </joint>
   <link name="arm1">
@@ -87,5 +88,5 @@
     </inertial>
   </link>
-  <joint name="joint2" type="continuous">
+  <joint name="joint1" type="continuous">
     <!-- -pi rotation so that for 0 pendulum is downward -->
     <origin xyz="${arm1_length} 0.0 0.0" rpy="${-pi} 0.0 0.0" />
@@ -94,5 +95,5 @@
     <axis xyz="1 0 0" />
     <dynamics damping="$(arg b2)" />
-    <limit effort="${max_effort}" velocity="${max_velocity}" />
+    <limit effort="${max_effort}" velocity="${max_velocity_joint1}" />
   </joint>
   <link name="arm2">
@@ -124,5 +125,5 @@
       </xacro:if>
     </hardware>
-    <joint name="joint1">
+    <joint name="joint0">
       <command_interface name="effort">
         <param name="min">${-max_effort}</param>
@@ -132,5 +133,5 @@
       <state_interface name="velocity" />
     </joint>
-    <joint name="joint2">
+    <joint name="joint1">
       <command_interface name="effort">
         <param name="min">${-max_effort}</param>

File: furuta_pendulum_drake/urdf/furuta_pendulum.urdf (robot description, URDF)
Before this commit: robot furuta_pendulum, 4 links, 3 joints
Joints:
- removed joint joint2
- added joint joint0: type continuous, parent base_link, child arm1, origin xyz=0.0 0.0 0.184 rpy=0.0 0.0 0.0, axis 0 0 1, limit effort=4.0 velocity=15.0
- joint joint1: axis 0 0 1 -> 1 0 0; child arm1 -> arm2; origin xyz=0.0 0.0 0.184 rpy=0.0 0.0 0.0 -> xyz=0.093525 0.0 0.0 rpy=-3.141592653589793 0.0 0.0; parent base_link -> arm1

File: furuta_pendulum_hardware/urdf/furuta_pendulum.urdf.xacro (robot description, xacro)
@@ -57,5 +57,5 @@
     </inertial>
   </link>
-  <joint name="joint1" type="continuous">
+  <joint name="joint0" type="continuous">
     <origin xyz="0.0 0.0 ${base_length+arm1_radius}" rpy="0.0 0.0 0.0" />
     <parent link="base_link" />
@@ -87,5 +87,5 @@
     </inertial>
   </link>
-  <joint name="joint2" type="continuous">
+  <joint name="joint1" type="continuous">
     <!-- -pi rotation so that for 0 pendulum is downward -->
     <origin xyz="${arm1_length} 0.0 0.0" rpy="${-pi} 0.0 0.0" />

File: furuta_pendulum_rl/model/furuta_pendulum.urdf (robot description, URDF)
Before this commit: robot furuta_pendulum, 3 links, 2 joints
Joints:
- removed joint joint2
- added joint joint0: type continuous, parent base_link, child arm1, origin xyz=0.0 0.0 0.184 rpy=0.0 0.0 0.0, axis 0 0 1, limit effort=4.0 velocity=15.0
- joint joint1: axis 0 0 1 -> 1 0 0; child arm1 -> arm2; origin xyz=0.0 0.0 0.184 rpy=0.0 0.0 0.0 -> xyz=0.093525 0.0 0.0 rpy=-3.141592653589793 0.0 0.0; parent base_link -> arm1
