Commit message: Change pendulum bodies size

File: furuta_pendulum_description/urdf/furuta_pendulum.urdf.xacro (robot description, xacro)
@@ -15,10 +15,10 @@
     <color rgba="0.8 0.8 0.8 1.0" />
   </material>
-  <xacro:property name="base_radius" value="0.1" />
+  <xacro:property name="base_radius" value="0.025" />
   <xacro:property name="L2" value="$(arg L2)" />
   <xacro:property name="base_length" value="${L2+0.05}" />
-  <xacro:property name="arm1_radius" value="0.02" />
+  <xacro:property name="arm1_radius" value="0.005" />
   <xacro:property name="arm1_length" value="$(arg L1)" />
-  <xacro:property name="arm2_radius" value="0.02" />
+  <xacro:property name="arm2_radius" value="0.005" />
   <xacro:property name="arm2_length" value="$(arg L2)" />
   <!-- https://www.hindawi.com/journals/jcse/2011/528341/ here this inertias

Commit message: Update urdf

File: furuta_pendulum_description/urdf/furuta_pendulum.urdf.xacro (robot description, xacro)
@@ -27,6 +27,6 @@
   <xacro:property name="arm1_inertia_x" value="0.000001" />
   <xacro:property name="arm2_inertia_z" value="0.000001" />
-  <xacro:property name="max_effort" value="4.0" />
-  <xacro:property name="max_velocity_joint0" value="18.0" />
+  <xacro:property name="max_effort" value="0.43" />
+  <xacro:property name="max_velocity_joint0" value="22.0" />
   <xacro:property name="max_velocity_joint1" value="100.0" />
   <link name="world" />
